Commit message: refactor panda_arm.ros2_control.xacro to use a macro for configuring the joints

File: franka_description/robots/panda_arm.ros2_control.xacro (robot description, xacro)
@@ -14,60 +14,20 @@
         </xacro:unless>
       </hardware>
-      <joint name="${ns}_joint1">
-        <param name="initial_position">0.0</param>
-        <command_interface name="effort">
-        </command_interface>
-        <state_interface name="position"/>
-        <state_interface name="velocity"/>
-        <state_interface name="effort"/>
-      </joint>
-      <joint name="${ns}_joint2">
-        <param name="initial_position">-0.785</param>
-        <command_interface name="effort">
-        </command_interface>
-        <state_interface name="position"/>
-        <state_interface name="velocity"/>
-        <state_interface name="effort"/>
-      </joint>
-      <joint name="${ns}_joint3">
-        <param name="initial_position">0.0</param>
-        <command_interface name="effort">
-        </command_interface>
-        <state_interface name="position"/>
-        <state_interface name="velocity"/>
-        <state_interface name="effort"/>
-      </joint>
-      <joint name="${ns}_joint4">
-        <param name="initial_position">-2.356</param>
-        <command_interface name="effort">
-        </command_interface>
-        <state_interface name="position"/>
-        <state_interface name="velocity"/>
-        <state_interface name="effort"/>
-      </joint>
-      <joint name="${ns}_joint5">
-        <param name="initial_position">0.0</param>
-        <command_interface name="effort">
-        </command_interface>
-        <state_interface name="position"/>
-        <state_interface name="velocity"/>
-        <state_interface name="effort"/>
-      </joint>
-      <joint name="${ns}_joint6">
-        <param name="initial_position">1.571</param>
-        <command_interface name="effort">
-        </command_interface>
-        <state_interface name="position"/>
-        <state_interface name="velocity"/>
-        <state_interface name="effort"/>
-      </joint>
-      <joint name="${ns}_joint7">
-        <param name="initial_position">0.785</param>
-        <command_interface name="effort">
-        </command_interface>
-        <state_interface name="position"/>
-        <state_interface name="velocity"/>
-        <state_interface name="effort"/>
-      </joint>
+      <xacro:macro name="configure_joint" params="joint_name initial_position">
+        <joint name="${joint_name}">
+          <param name="initial_position">${initial_position}</param>
+          <command_interface name="effort"/>
+          <state_interface name="position"/>
+          <state_interface name="velocity"/>
+          <state_interface name="effort"/>
+        </joint>
+      </xacro:macro>
+      <xacro:configure_joint joint_name="${ns}_joint1" initial_position="0.0"/>
+      <xacro:configure_joint joint_name="${ns}_joint2" initial_position="-${pi/4}"/>
+      <xacro:configure_joint joint_name="${ns}_joint3" initial_position="0.0"/>
+      <xacro:configure_joint joint_name="${ns}_joint4" initial_position="${-3*pi/4}"/>
+      <xacro:configure_joint joint_name="${ns}_joint5" initial_position="0.0"/>
+      <xacro:configure_joint joint_name="${ns}_joint6" initial_position="${pi/2}"/>
+      <xacro:configure_joint joint_name="${ns}_joint7" initial_position="${pi/4}"/>
     </ros2_control>
   </xacro:macro>

Commit message: use pi to generate predefined moveit poses

File: franka_description/robots/panda_arm.ros2_control.xacro (robot description, xacro)
@@ -24,5 +24,5 @@
       </xacro:macro>
       <xacro:configure_joint joint_name="${ns}_joint1" initial_position="0.0"/>
-      <xacro:configure_joint joint_name="${ns}_joint2" initial_position="-${pi/4}"/>
+      <xacro:configure_joint joint_name="${ns}_joint2" initial_position="${-pi/4}"/>
       <xacro:configure_joint joint_name="${ns}_joint3" initial_position="0.0"/>
       <xacro:configure_joint joint_name="${ns}_joint4" initial_position="${-3*pi/4}"/>

File: franka_moveit_config/srdf/panda_arm.xacro (robot description, xacro)
@@ -7,10 +7,10 @@
     <group_state name="ready" group="${arm_id}_arm">
       <joint name="${arm_id}_joint1" value="0"/>
-      <joint name="${arm_id}_joint2" value="-0.785"/>
+      <joint name="${arm_id}_joint2" value="${-pi/4}"/>
       <joint name="${arm_id}_joint3" value="0"/>
-      <joint name="${arm_id}_joint4" value="-2.356"/>
+      <joint name="${arm_id}_joint4" value="${-3*pi/4}"/>
       <joint name="${arm_id}_joint5" value="0"/>
-      <joint name="${arm_id}_joint6" value="1.571"/>
-      <joint name="${arm_id}_joint7" value="0.785"/>
+      <joint name="${arm_id}_joint6" value="${pi/2}"/>
+      <joint name="${arm_id}_joint7" value="${pi/4}"/>
     </group_state>
     <group_state name="extended" group="${arm_id}_arm">
@@ -20,6 +20,6 @@
       <joint name="${arm_id}_joint4" value="-0.1"/>
       <joint name="${arm_id}_joint5" value="0"/>
-      <joint name="${arm_id}_joint6" value="1.571"/>
-      <joint name="${arm_id}_joint7" value="0.785"/>
+      <joint name="${arm_id}_joint6" value="${pi/2}"/>
+      <joint name="${arm_id}_joint7" value="${pi/4}"/>
     </group_state>
     <virtual_joint name="virtual_joint" type="fixed" parent_frame="world" child_link="${arm_id}_link0"/>
