Commit message: add panda_hand_tcp to franka_description

File: franka_description/robots/hand.xacro (robot description, xacro)
@@ -19,5 +19,5 @@
         <origin xyz="0 0 0.04" rpy="0 ${pi/2} ${pi/2}"/>
         <geometry>
-          <cylinder radius="${0.04+safety_distance}" length="0.1" />
+          <cylinder radius="${0.04+safety_distance}" length="0.1"/>
         </geometry>
       </collision>
@@ -25,5 +25,5 @@
         <origin xyz="0 -0.05 0.04" rpy="0 0 0"/>
         <geometry>
-          <sphere radius="${0.04+safety_distance}"  />
+          <sphere radius="${0.04+safety_distance}"/>
         </geometry>
       </collision>
@@ -31,5 +31,5 @@
         <origin xyz="0 0.05 0.04" rpy="0 0 0"/>
         <geometry>
-          <sphere radius="${0.04+safety_distance}"  />
+          <sphere radius="${0.04+safety_distance}"/>
         </geometry>
       </collision>
@@ -37,5 +37,5 @@
         <origin xyz="0 0 0.1" rpy="0 ${pi/2} ${pi/2}"/>
         <geometry>
-          <cylinder radius="${0.02+safety_distance}" length="0.1" />
+          <cylinder radius="${0.02+safety_distance}" length="0.1"/>
         </geometry>
       </collision>
@@ -43,5 +43,5 @@
         <origin xyz="0 -0.05 0.1" rpy="0 0 0"/>
         <geometry>
-          <sphere radius="${0.02+safety_distance}"  />
+          <sphere radius="${0.02+safety_distance}"/>
         </geometry>
       </collision>
@@ -49,8 +49,15 @@
         <origin xyz="0 0.05 0.1" rpy="0 0 0"/>
         <geometry>
-          <sphere radius="${0.02+safety_distance}"  />
+          <sphere radius="${0.02+safety_distance}"/>
         </geometry>
       </collision>
     </link>
+    <!-- Define the hand_tcp frame -->
+    <link name="${ns}_hand_tcp"/>
+    <joint name="${ns}_hand_tcp_joint" type="fixed">
+      <origin xyz="0 0 0.1034" rpy="0 0 0"/>
+      <parent link="${ns}_hand"/>
+      <child link="${ns}_hand_tcp"/>
+    </joint>
     <link name="${ns}_leftfinger">
       <visual>
@@ -67,5 +74,5 @@
         </geometry>
       </visual>
-   </link>
+    </link>
     <joint name="${ns}_finger_joint1" type="prismatic">
       <parent link="${ns}_hand"/>
@@ -81,5 +88,5 @@
       <axis xyz="0 -1 0"/>
       <limit effort="20" lower="0.0" upper="0.04" velocity="0.2"/>
-      <mimic joint="${ns}_finger_joint1" />
+      <mimic joint="${ns}_finger_joint1"/>
     </joint>
   </xacro:macro>
