Commit message: first version of franka_hardware

File: franka_description/robots/panda_arm.urdf.xacro (robot description, xacro)
@@ -4,5 +4,11 @@
   <xacro:arg name="hand"   default="false" /> <!-- Should a franka_gripper be mounted at the flange?" -->
   <xacro:arg name="gazebo" default="false" /> <!-- Is the robot being simulated in gazebo?" -->
+  <xacro:arg name="robot_ip" default="franka" /> <!-- IP address or hostname of the robot" -->
+  <xacro:arg name="use_fake_hardware" default="false"/>
+  <xacro:arg name="fake_sensor_commands" default="false"/>
   <xacro:property name="arm_id" value="$(arg arm_id)" />
+  <xacro:property name="robot_ip" value="$(arg robot_ip)" />
+  <xacro:property name="use_fake_hardware" value="$(arg use_fake_hardware)" />
+  <xacro:property name="fake_sensor_commands" value="$(arg fake_sensor_commands)" />
   <xacro:unless value="$(arg gazebo)">
     <!-- Create a URDF for a real hardware -->
@@ -13,4 +19,6 @@
       <xacro:hand ns="${arm_id}" rpy="0 0 ${-pi/4}" connected_to="${arm_id}_link8" safety_distance="0.03"/>
     </xacro:if>
+    <xacro:include filename="$(find franka_description)/robots/panda_arm.ros2_control.xacro"/>
+    <xacro:panda_arm_ros2_control ns="${arm_id}" robot_ip="${robot_ip}" use_fake_hardware="${use_fake_hardware}" fake_sensor_commands="${fake_sensor_commands}"/>
   </xacro:unless>
   <xacro:if value="$(arg gazebo)">

Commit message: remove gazebo and dual arm urdf files from franka_description

File: franka_description/robots/panda_arm.urdf.xacro (robot description, xacro)
@@ -1,64 +1,16 @@
 <?xml version='1.0' encoding='utf-8'?>
 <robot xmlns:xacro="http://www.ros.org/wiki/xacro" name="panda">
-  <xacro:arg name="arm_id" default="panda" /> <!-- Name of this panda -->
-  <xacro:arg name="hand"   default="false" /> <!-- Should a franka_gripper be mounted at the flange?" -->
-  <xacro:arg name="gazebo" default="false" /> <!-- Is the robot being simulated in gazebo?" -->
-  <xacro:arg name="robot_ip" default="" /> <!-- IP address or hostname of the robot" -->
+  <xacro:arg name="arm_id" default="panda"/> <!-- Name of this panda -->
+  <xacro:arg name="hand" default="false"/> <!-- Should a franka_gripper be mounted at the flange?" -->
+  <xacro:arg name="robot_ip" default=""/> <!-- IP address or hostname of the robot" -->
   <xacro:arg name="use_fake_hardware" default="false"/>
   <xacro:arg name="fake_sensor_commands" default="false"/>
-  <xacro:property name="arm_id" value="$(arg arm_id)" />
-  <xacro:property name="robot_ip" value="$(arg robot_ip)" />
-  <xacro:property name="use_fake_hardware" value="$(arg use_fake_hardware)" />
-  <xacro:property name="fake_sensor_commands" value="$(arg fake_sensor_commands)" />
-  <xacro:unless value="$(arg gazebo)">
-    <!-- Create a URDF for a real hardware -->
-    <xacro:include filename="$(find franka_description)/robots/panda_arm.xacro" />
-    <xacro:panda_arm arm_id="${arm_id}" safety_distance="0.03"/>
-    <xacro:if value="$(arg hand)">
-      <xacro:include filename="$(find franka_description)/robots/hand.xacro"/>
-      <xacro:hand ns="${arm_id}" rpy="0 0 ${-pi/4}" connected_to="${arm_id}_link8" safety_distance="0.03"/>
-    </xacro:if>
-    <xacro:include filename="$(find franka_description)/robots/panda_arm.ros2_control.xacro"/>
-    <xacro:panda_arm_ros2_control ns="${arm_id}" robot_ip="${robot_ip}" use_fake_hardware="${use_fake_hardware}" fake_sensor_commands="${fake_sensor_commands}"/>
-  </xacro:unless>
-  <xacro:if value="$(arg gazebo)">
-    <xacro:arg name="xyz" default="0 0 0" />
-    <xacro:arg name="rpy" default="0 0 0" />
-    <!-- Create a simulatable URDF -->
-    <xacro:include filename="$(find franka_description)/robots/utils.xacro" />
-    <xacro:include filename="$(find franka_description)/robots/panda_gazebo.xacro" />
-    <xacro:panda_arm arm_id="${arm_id}" />
-    <xacro:if value="$(arg hand)">
-      <xacro:hand ns="${arm_id}" rpy="0 0 ${-pi/4}" connected_to="${arm_id}_link8" />
-      <xacro:gazebo-joint joint="${arm_id}_finger_joint1" transmission="hardware_interface/EffortJointInterface" />
-      <xacro:gazebo-joint joint="${arm_id}_finger_joint2" transmission="hardware_interface/EffortJointInterface" />
-    </xacro:if>
-    <!-- Gazebo requires a joint to a link called "world" for statically mounted robots -->
-    <link name="world" />
-    <joint name="world_joint" type="fixed">
-      <origin xyz="$(arg xyz)" rpy="$(arg rpy)" />
-      <parent link="world" />
-      <child  link="${arm_id}_link0" />
-    </joint>
-    <xacro:gazebo-joint joint="${arm_id}_joint1" transmission="hardware_interface/EffortJointInterface" />
-    <xacro:gazebo-joint joint="${arm_id}_joint2" transmission="hardware_interface/EffortJointInterface" />
-    <xacro:gazebo-joint joint="${arm_id}_joint3" transmission="hardware_interface/EffortJointInterface" />
-    <xacro:gazebo-joint joint="${arm_id}_joint4" transmission="hardware_interface/EffortJointInterface" />
-    <xacro:gazebo-joint joint="${arm_id}_joint5" transmission="hardware_interface/EffortJointInterface" />
-    <xacro:gazebo-joint joint="${arm_id}_joint6" transmission="hardware_interface/EffortJointInterface" />
-    <xacro:gazebo-joint joint="${arm_id}_joint7" transmission="hardware_interface/EffortJointInterface" />
-    <xacro:transmission-franka-state arm_id="${arm_id}" />
-    <xacro:transmission-franka-model arm_id="${arm_id}"
-       root="${arm_id}_joint1"
-       tip="${arm_id}_joint8"
-     />
-    <gazebo>
-      <plugin name="gazebo_ros_control" filename="libgazebo_ros_control.so">
-        <robotNamespace>${arm_id}</robotNamespace>
-        <controlPeriod>0.001</controlPeriod>
-        <robotSimType>franka_gazebo/FrankaHWSim</robotSimType>
-      </plugin>
-      <self_collide>true</self_collide>
-    </gazebo>
+  <xacro:include filename="$(find franka_description)/robots/panda_arm.xacro"/>
+  <xacro:panda_arm arm_id="$(arg arm_id)" safety_distance="0.03"/>
+  <xacro:if value="$(arg hand)">
+    <xacro:include filename="$(find franka_description)/robots/hand.xacro"/>
+    <xacro:hand ns="$(arg arm_id)" rpy="0 0 ${-pi/4}" connected_to="$(arg arm_id)_link8" safety_distance="0.03"/>
   </xacro:if>
+  <xacro:include filename="$(find franka_description)/robots/panda_arm.ros2_control.xacro"/>
+  <xacro:panda_arm_ros2_control ns="$(arg arm_id)" robot_ip="$(arg robot_ip)" use_fake_hardware="$(arg use_fake_hardware)" fake_sensor_commands="$(arg fake_sensor_commands)"/>
 </robot>

Commit message: Added support for Ignition
Signed-off-by: ahcorde <ahcorde@gmail.com>

File: franka_description/robots/panda_arm.urdf.xacro (robot description, xacro)
@@ -6,11 +6,25 @@
   <xacro:arg name="use_fake_hardware" default="false"/>
   <xacro:arg name="fake_sensor_commands" default="false"/>
+  <xacro:arg name="ignition_sim" default="true"/>
   <xacro:include filename="$(find franka_description)/robots/panda_arm.xacro"/>
-  <xacro:panda_arm arm_id="$(arg arm_id)" safety_distance="0.03"/>
+  <!-- Used for fixing robot to Gazebo 'base_link' -->
+  <xacro:if value="$(arg ignition_sim)">
+    <link name="world"/>
+    <xacro:panda_arm arm_id="$(arg arm_id)" safety_distance="0.03" connected_to="world"/>
+  </xacro:if>
+  <xacro:unless value="$(arg ignition_sim)">
+    <xacro:panda_arm arm_id="$(arg arm_id)" safety_distance="0.03"/>
+  </xacro:unless>
   <xacro:if value="$(arg hand)">
     <xacro:include filename="$(find franka_description)/robots/hand.xacro"/>
     <xacro:hand ns="$(arg arm_id)" rpy="0 0 ${-pi/4}" connected_to="$(arg arm_id)_link8" safety_distance="0.03"/>
   </xacro:if>
-  <xacro:include filename="$(find franka_description)/robots/panda_arm.ros2_control.xacro"/>
-  <xacro:panda_arm_ros2_control ns="$(arg arm_id)" robot_ip="$(arg robot_ip)" use_fake_hardware="$(arg use_fake_hardware)" fake_sensor_commands="$(arg fake_sensor_commands)"/>
+  <xacro:if value="$(arg ignition_sim)">
+    <xacro:include filename="$(find franka_description)/robots/panda_arm.ignition.xacro"/>
+    <xacro:panda_arm_ignition ns="$(arg arm_id)"/>
+  </xacro:if>
+  <xacro:unless value="$(arg ignition_sim)">
+    <xacro:include filename="$(find franka_description)/robots/panda_arm.ros2_control.xacro"/>
+    <xacro:panda_arm_ros2_control ns="$(arg arm_id)" robot_ip="$(arg robot_ip)" use_fake_hardware="$(arg use_fake_hardware)" fake_sensor_commands="$(arg fake_sensor_commands)"/>
+  </xacro:unless>
 </robot>
