Commit message: adapt extended gripper pose

File: franka_moveit_config/srdf/panda_arm.xacro (robot description, xacro)
@@ -18,5 +18,5 @@
       <joint name="${arm_id}_joint2" value="0"/>
       <joint name="${arm_id}_joint3" value="0"/>
-      <joint name="${arm_id}_joint4" value="0"/>
+      <joint name="${arm_id}_joint4" value="-0.1"/>
       <joint name="${arm_id}_joint5" value="0"/>
       <joint name="${arm_id}_joint6" value="1.571"/>

Commit message: add panda_manipulator move-group

File: franka_moveit_config/srdf/panda_arm.xacro (robot description, xacro)
@@ -2,25 +2,7 @@
 <robot xmlns:xacro="http://www.ros.org/wiki/xacro" name="panda">
   <xacro:macro name="panda_arm" params="arm_id:='panda' ">
-    <group name="${arm_id}_arm">
-      <chain base_link="${arm_id}_link0" tip_link="${arm_id}_link8"/>
-    </group>
-    <group_state name="ready" group="${arm_id}_arm">
-      <joint name="${arm_id}_joint1" value="0"/>
-      <joint name="${arm_id}_joint2" value="${-pi/4}"/>
-      <joint name="${arm_id}_joint3" value="0"/>
-      <joint name="${arm_id}_joint4" value="${-3*pi/4}"/>
-      <joint name="${arm_id}_joint5" value="0"/>
-      <joint name="${arm_id}_joint6" value="${pi/2}"/>
-      <joint name="${arm_id}_joint7" value="${pi/4}"/>
-    </group_state>
-    <group_state name="extended" group="${arm_id}_arm">
-      <joint name="${arm_id}_joint1" value="0"/>
-      <joint name="${arm_id}_joint2" value="0"/>
-      <joint name="${arm_id}_joint3" value="0"/>
-      <joint name="${arm_id}_joint4" value="-0.1"/>
-      <joint name="${arm_id}_joint5" value="0"/>
-      <joint name="${arm_id}_joint6" value="${pi/2}"/>
-      <joint name="${arm_id}_joint7" value="${pi/4}"/>
-    </group_state>
+    <xacro:include filename="$(find franka_moveit_config)/srdf/arm.xacro"/>
+    <xacro:arm arm_id="${arm_id}" group_name="${arm_id}_manipulator" tip_link="${arm_id}_hand_tcp"/>
+    <xacro:arm arm_id="${arm_id}" group_name="${arm_id}_arm" tip_link="${arm_id}_link8"/>
     <virtual_joint name="virtual_joint" type="fixed" parent_frame="world" child_link="${arm_id}_link0"/>
     <disable_collisions link1="${arm_id}_link0" link2="${arm_id}_link1" reason="Adjacent"/>

File: franka_moveit_config/srdf/panda_arm_hand.xacro (robot description, xacro)
@@ -2,8 +2,4 @@
 <robot xmlns:xacro="http://www.ros.org/wiki/xacro" name="panda">
   <xacro:macro name="panda_arm_hand" params="arm_id:='panda' ">
-    <group name="${arm_id}_arm_hand">
-      <group name="${arm_id}_arm"/>
-      <group name="hand"/>
-    </group>
     <group_state name="open" group="hand">
       <joint name="${arm_id}_finger_joint1" value="0.035"/>
@@ -14,4 +10,5 @@
       <joint name="${arm_id}_finger_joint2" value="0"/>
     </group_state>
+    <end_effector name="hand_tcp" parent_link="${arm_id}_hand_tcp" group="hand" parent_group="${arm_id}_manipulator"/>
     <end_effector name="hand" parent_link="${arm_id}_link8" group="hand" parent_group="${arm_id}_arm"/>
     <disable_collisions link1="${arm_id}_hand" link2="${arm_id}_link3" reason="Never"/>
