Commit message: rename arm.xacro to group_definition.xacro

File: franka_moveit_config/srdf/group_definition.xacro (robot description, xacro)
@@ -1,5 +1,5 @@
 <?xml version="1.0" encoding="UTF-8"?>
 <robot xmlns:xacro="http://www.ros.org/wiki/xacro" name="panda">
-  <xacro:macro name="arm" params="group_name arm_id tip_link">
+  <xacro:macro name="group_definition" params="group_name arm_id tip_link">
     <group name="${group_name}">
       <chain base_link="${arm_id}_link0" tip_link="${tip_link}"/>

File: franka_moveit_config/srdf/panda_arm.xacro (robot description, xacro)
@@ -2,7 +2,7 @@
 <robot xmlns:xacro="http://www.ros.org/wiki/xacro" name="panda">
   <xacro:macro name="panda_arm" params="arm_id:='panda' ">
-    <xacro:include filename="$(find franka_moveit_config)/srdf/arm.xacro"/>
-    <xacro:arm arm_id="${arm_id}" group_name="${arm_id}_manipulator" tip_link="${arm_id}_hand_tcp"/>
-    <xacro:arm arm_id="${arm_id}" group_name="${arm_id}_arm" tip_link="${arm_id}_link8"/>
+    <xacro:include filename="$(find franka_moveit_config)/srdf/group_definition.xacro"/>
+    <xacro:group_definition arm_id="${arm_id}" group_name="${arm_id}_manipulator" tip_link="${arm_id}_hand_tcp"/>
+    <xacro:group_definition arm_id="${arm_id}" group_name="${arm_id}_arm" tip_link="${arm_id}_link8"/>
     <virtual_joint name="virtual_joint" type="fixed" parent_frame="world" child_link="${arm_id}_link0"/>
     <disable_collisions link1="${arm_id}_link0" link2="${arm_id}_link1" reason="Adjacent"/>
